Commit message: success in simple loco-manipulation

File: loco_manipulation_gym/resources/robots/tita_noarm/robots.urdf (robot description, URDF)
Before this commit: robot tita, 17 links, 16 joints
Joints:
- joint left_ankle: limit lower=-999999 upper=999999 effort=15 velocity=20 -> lower=-6.283185e4 upper=6.283185e4 effort=100 velocity=100
- joint right_ankle: limit lower=-999999 upper=999999 effort=15 velocity=20 -> lower=-6.283185e4 upper=6.283185e4 effort=100 velocity=100
