Commit message: update base orientation limits

File: loco_manipulation_gym/resources/robots/tita_simple/tita_simple.urdf (robot description, URDF)
Before this commit: robot tita_arx, 17 links, 16 joints
Links:
- added link virtual_base, mass 0.5
Joints:
- removed joint floating_base
- added joint base_motion: type planar, parent world, child virtual_base, axis 1 0 0, limit lower=-100 upper=100 effort=100 velocity=100
- added joint base_to_virtual: type fixed, parent virtual_base, child base_link, origin xyz=0 0 0 rpy=0 0 0
- joint left_ankle: axis 0 0 1 -> (none); limit lower=-6.283185e4 upper=6.283185e4 effort=100 velocity=100 -> (none); type revolute -> fixed
- joint left_hip: axis 0 0 1 -> (none); limit lower=-1.919862 upper=3.490659 effort=100 velocity=100 -> (none); origin xyz=0.1426 0 0 rpy=-1.5708 0 -1.5708 -> xyz=0.1426 0 0 rpy=-1.5708 0 -0.7708; type revolute -> fixed
- joint left_knee: axis 0 0 1 -> (none); limit lower=-2.670354 upper=-0.698132 effort=100 velocity=100 -> (none); origin xyz=0.2 0 0 rpy=0 0 0 -> xyz=0.2 0 0 rpy=0 0 -1.5; type revolute -> fixed
- joint right_ankle: axis 0 0 1 -> (none); limit lower=-6.283185e4 upper=6.283185e4 effort=100 velocity=100 -> (none); type revolute -> fixed
- joint right_hip: axis 0 0 1 -> (none); limit lower=-1.919862 upper=3.490659 effort=100 velocity=100 -> (none); origin xyz=-0.1426 0 0 rpy=-1.5708 0 -1.5708 -> xyz=-0.1426 0 0 rpy=-1.5708 0 -0.7708; type revolute -> fixed
- joint right_knee: axis 0 0 1 -> (none); limit lower=-2.670354 upper=-0.698132 effort=100 velocity=100 -> (none); origin xyz=0.2 0 0 rpy=0 0 0 -> xyz=0.2 0 0 rpy=0 0 -1.5; type revolute -> fixed

File: loco_manipulation_gym/resources/robots/tita_simple/urdf/tita_arx-old.urdf (robot description, URDF)
Before this commit: robot tita_arx, 17 links, 16 joints
Links:
- link arm_link00: mass 0.44038 -> 0.422721353715926
- link arm_link01: mass 0.060835 -> 0.0968040209395549
- link arm_link02: mass 1.0733 -> 1.11872105871019
- link arm_link03: mass 0.4994 -> 0.840824525877169
- link arm_link04: mass 0.080971 -> 0.124324803309629
- link arm_link05: mass 0.60236 -> 0.636013398718113
- link gripper_link: mass 0.6000 -> 0.562622175728676
Joints:
- joint arm_joint00: origin xyz=0 0 0.0603 rpy=0 0 0 -> xyz=0 0 0.0565 rpy=0 0 0
- joint arm_joint01: origin xyz=0.02 0 0.0402 rpy=0 0 0 -> xyz=0.02 0 0.047 rpy=0 0 0
- joint arm_joint03: origin xyz=0.245 0 -0.056 rpy=0 0 0 -> xyz=0.245 -5E-05 -0.06 rpy=0 0 0
- joint arm_joint04: origin xyz=0.06575 -0.001 -0.0825 rpy=0 0 0 -> xyz=0.073914 5E-05 -0.083391 rpy=0 0 0
- joint arm_joint05: origin xyz=0.02845 0 0.0825 rpy=-3.1416 0 0 -> xyz=0.025286 0 0.083391 rpy=3.1416 0 0
- joint trunk_arm_joint_base_0: origin xyz=0.0 0 0.1 rpy=0 0 0 -> xyz=0.018 0 0.072 rpy=0 0 0

File: loco_manipulation_gym/resources/robots/tita_simple/urdf/tita_simple.urdf (robot description, URDF)
Before this commit: robot tita_arx, 17 links, 16 joints
Joints:
- joint floating_base: origin xyz=0 0 0 rpy=0 0 0 -> (none)
- joint left_ankle: axis 0 0 1 -> (none); limit lower=-6.283185e4 upper=6.283185e4 effort=100 velocity=100 -> (none); type revolute -> fixed
- joint left_hip: axis 0 0 1 -> (none); limit lower=-1.919862 upper=3.490659 effort=100 velocity=100 -> (none); origin xyz=0.1426 0 0 rpy=-1.5708 0 -1.5708 -> xyz=0.1426 0 0 rpy=-1.5708 0 -0.7708; type revolute -> fixed
- joint left_knee: axis 0 0 1 -> (none); limit lower=-2.670354 upper=-0.698132 effort=100 velocity=100 -> (none); origin xyz=0.2 0 0 rpy=0 0 0 -> xyz=0.2 0 0 rpy=0 0 -1.5; type revolute -> fixed
- joint right_ankle: axis 0 0 1 -> (none); limit lower=-6.283185e4 upper=6.283185e4 effort=100 velocity=100 -> (none); type revolute -> fixed
- joint right_hip: axis 0 0 1 -> (none); limit lower=-1.919862 upper=3.490659 effort=100 velocity=100 -> (none); origin xyz=-0.1426 0 0 rpy=-1.5708 0 -1.5708 -> xyz=-0.1426 0 0 rpy=-1.5708 0 -0.7708; type revolute -> fixed
- joint right_knee: axis 0 0 1 -> (none); limit lower=-2.670354 upper=-0.698132 effort=100 velocity=100 -> (none); origin xyz=0.2 0 0 rpy=0 0 0 -> xyz=0.2 0 0 rpy=0 0 -1.5; type revolute -> fixed
